File: Eagle/BinaryClockDisplay.brd (EAGLE design)
At the start: 75.9 x 59.7 mm, 43 parts

Commit message: Adjusted schematics and circuit-board
Parts:
- moved S1 68.8 mm to (68.5, 63.5), flipped to the top
- moved JP3 43.4 mm to (46.9, 23.7), flipped to the bottom, turned to 90 degrees
- moved JP2 3.61 mm to (38.7, 64.0)
Connections:
- net GND: now also JP2.2
Routing:
- net GND: track 529.3 -> 642.1 mm, vias 0 -> 1
- net N$3: track 22.1 -> 77.0 mm
- net N$2: track 16.9 -> 66.5 mm
- net N$4: track 26.2 -> 58.6 mm
- net GPIO11: track 56.8 -> 29.3 mm
- net +3V3: track 369.7 -> 358.9 mm
- net GPIO9: track 78.9 -> 79.9 mm

Commit message: Circuitboard as ordered from Aisler 2019-02-03
Also a
Parts:
- moved S1 75.4 mm to (13.3, 12.1), flipped to the bottom, turned to 180 degrees
Connections:
- removed net +3V3: C1.1, C10.1, C11.1, C12.1, C13.1, C14.1, C15.1, C16.1, C17.1, C18.1, C19.1, C2.1, C20.1, C3.1, C4.1, C5.1, C6.1, C7.1, C8.1, C9.1, D1.1, D10.1, D11.1, D12.1, D13.1, D14.1, D15.1, D16.1, D17.1, D18.1, D19.1, D2.1, D20.1, D3.1, D4.1, D5.1, D6.1, D7.1, D8.1, D9.1, JP2.1, JP3.1
- removed net GPIO9: D1.4, JP2.21
- new net 5V: C1.1, C10.1, C11.1, C12.1, C13.1, C14.1, C15.1, C16.1, C17.1, C18.1, C19.1, C2.1, C20.1, C3.1, C4.1, C5.1, C6.1, C7.1, C8.1, C9.1, D1.1, D10.1, D11.1, D12.1, D13.1, D14.1, D15.1, D16.1, D17.1, D18.1, D19.1, D2.1, D20.1, D3.1, D4.1, D5.1, D6.1, D7.1, D8.1, D9.1, JP2.2
- new net GPIO18: D1.4, JP2.12
- net GND: now also JP2.6; no longer JP2.2
Routing:
- net 5V: track 0.00 -> 361.2 mm, vias 0 -> 20
- net +3V3: track 358.9 -> 0.00 mm, vias 20 -> 0
- net GPIO11: track 29.3 -> 138.0 mm
- net GPIO18: track 0.00 -> 95.6 mm
- net GPIO9: track 79.9 -> 0.00 mm
- net GND: track 642.1 -> 664.7 mm
