File: Eagle/BinaryClockDisplay.brd (EAGLE design)
At the start: 75.9 x 59.7 mm, 44 parts

Commit message: Cleaning out some unused files
Parts:
- added JP4: IO, pinhead:1X05
- moved JP2 2.94 mm to (41.5, 64.9)
Connections:
- new net GPIO13: JP2.33, JP4.2
- new net GPIO19: JP2.35, JP4.3
- new net GPIO26: JP2.37, JP4.4
- new net GPIO6: JP2.31, JP4.1
- net GND: now also JP4.5
Routing:
- net GND: track 733.2 -> 768.8 mm
- net GPIO6: track 0.00 -> 23.2 mm
- net GPIO13: track 0.00 -> 19.6 mm
- net GPIO19: track 0.00 -> 16.0 mm
- net GPIO26: track 0.00 -> 12.4 mm
- net N$3: track 77.0 -> 70.7 mm
- net GPIO11: track 138.0 -> 144.3 mm
- net 5V: track 381.0 -> 387.2 mm
- net N$2: track 66.6 -> 68.0 mm
- net GPIO18: track 95.6 -> 96.1 mm
Other:
- board text added: "0/1"
- board text added: "0/2"
- board text added: "0/4"
- board text added: "0/8"
- board text added: "GPIO13"
- board text added: "GPIO19"
- board text added: "GPIO26"
- board text added: "GPIO6"
- board text added: "I/O"

Commit message: More fix and a temperature check turning off the pi  if too hot
Parts:
- moved JP2 2.51 mm to (39.0, 64.7)
Routing:
- net GND: track 768.8 -> 709.9 mm
- net 5V: track 387.2 -> 382.8 mm
- net GPIO26: track 12.4 -> 14.8 mm
- net GPIO19: track 16.0 -> 18.4 mm
- net GPIO13: track 19.6 -> 22.0 mm
- net GPIO6: track 23.2 -> 25.6 mm
- net N$3: track 70.7 -> 72.6 mm
- net N$4: track 58.8 -> 60.3 mm
- net 3V3: track 74.3 -> 75.1 mm
- net N$2: track 68.0 -> 68.7 mm

Commit message: HW version 2 allmost done...
Parts:
- added S2, S3: SWITCH, SparkFun-Electromechanical:TACTILE-SWITCH-1101NE
- moved S1 22.2 mm to (35.5, 11.9)
Connections:
- new net GPIO10: JP2.19, S3.2
- new net GPIO9: JP2.21, S2.2
- net GND: now also S2.1, S3.1
Routing:
- net GPIO10: track 0.00 -> 132.1 mm
- net GPIO9: track 0.00 -> 121.6 mm
- net GPIO11: track 144.4 -> 112.0 mm
- net GND: track 709.9 -> 683.0 mm
- net 3V3: track 75.1 -> 71.3 mm
Other:
- board text added: "F1 Set"
- board text added: "F2 Pair"
- board text added: "F3 Reset"
- board text removed: "Reset"
- board text removed: "The PyBinaryClock!"
