File: Eagle/BinaryClockDisplay.sch (EAGLE design)
At the start: 43 parts

Commit message: Adjusted schematics and circuit-board
Connections:
- net GND: now also JP2.2
Changed lines of the file:
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@@
 <part name="GND22" library="supply1" deviceset="GND" device=""/>
 <part name="GND23" library="supply1" deviceset="GND" device=""/>
+<part name="GND24" library="supply1" deviceset="GND" device=""/>
 </parts>
 <sheets>
@@
 <attribute name="VALUE" x="195.58" y="-7.62" size="1.778" layer="96"/>
 </instance>
+<instance part="GND24" gate="1" x="226.06" y="43.18" smashed="yes">
+<attribute name="VALUE" x="223.52" y="40.64" size="1.778" layer="96"/>
+</instance>
 </instances>
 <busses>
@@
 <wire x1="210.82" y1="-2.54" x2="198.12" y2="-2.54" width="0.1524" layer="91"/>
 </segment>
+<segment>
+<pinref part="JP2" gate="A" pin="2"/>
+<pinref part="GND24" gate="1" pin="GND"/>
+<wire x1="218.44" y1="45.72" x2="226.06" y2="45.72" width="0.1524" layer="91"/>
+</segment>
 </net>

Commit message: Circuitboard as ordered from Aisler 2019-02-03
Also a
Connections:
- removed net +3V3: C1.1, C10.1, C11.1, C12.1, C13.1, C14.1, C15.1, C16.1, C17.1, C18.1, C19.1, C2.1, C20.1, C3.1, C4.1, C5.1, C6.1, C7.1, C8.1, C9.1, D1.VDD, D10.VDD, D11.VDD, D12.VDD, D13.VDD, D14.VDD, D15.VDD, D16.VDD, D17.VDD, D18.VDD, D19.VDD, D2.VDD, D20.VDD, D3.VDD, D4.VDD, D5.VDD, D6.VDD, D7.VDD, D8.VDD, D9.VDD, JP2.1, JP3.1
- removed net GPIO9: D1.DI, JP2.21
- new net 5V: C1.1, C10.1, C11.1, C12.1, C13.1, C14.1, C15.1, C16.1, C17.1, C18.1, C19.1, C2.1, C20.1, C3.1, C4.1, C5.1, C6.1, C7.1, C8.1, C9.1, D1.VDD, D10.VDD, D11.VDD, D12.VDD, D13.VDD, D14.VDD, D15.VDD, D16.VDD, D17.VDD, D18.VDD, D19.VDD, D2.VDD, D20.VDD, D3.VDD, D4.VDD, D5.VDD, D6.VDD, D7.VDD, D8.VDD, D9.VDD, JP2.2
- new net GPIO18: D1.DI, JP2.12
- net GND: now also JP2.6; no longer JP2.2
